File: Swept/sweepv2.kicad_pcb (KiCad board)
At the start: 2 copper layers, 216.9 x 86.9 mm, 51 parts, among them J1 AudioJack4dpb, J2 AudioJack4dpb, SW10 SW_Push, SW11 SW_Push, SW11_r1 SW_Push, SW12 SW_Push, SW12_r1 SW_Push, SW13_r1 SW_Push, SW14 SW_Push, SW15 SW_Push, SW15_r1 SW_Push, SW16 SW_Push, SW16_r1 SW_Push, SW17 SW_Push, SW17_r1 SW_Push, SW18 SW_Push, SW18_r1 SW_Push, SW2 SW_Push, SW20 SW_Push, SW20_r1 SW_Push, SW21 SW_Push, SW21_r1 SW_Push, SW2_r1 SW_Push, SW3 SW_Push, SW3_r1 SW_Push, SW4 SW_Push, SW4_r1 SW_Push, SW5 SW_Push, SW5_r1 SW_Push, SW6 SW_Push, SW6_r1 SW_Push, SW7_r1 SW_Push, SW8 SW_Push, SW8_r1 SW_Push, SW9 SW_Push, SW9_r1 SW_Push, U1 ProMicro-kbd, U2 ProMicro-kbd

Commit message: Schematic finished, pcb ready to route.
Parts:
- removed B+ (x2), B- (x2): MountingHole_Pad, kbd:1pin_conn
- removed G***: LOGO, Kailh:ferris_broom
- removed J1, J2: AudioJack4dpb, Kailh:TRRS-PJ-320A
- removed POWER SW: SW_SPDT, Kailh:SPDT_C128955 (x2)
- added Bat+1: MountingHole_Pad, kbd:1pin_conn, F.Cu at (20.6, 47.4)
- added Bat+r1: MountingHole_Pad, kbd:1pin_conn, F.Cu at (263.9, 47.6)
- added BatGND1: MountingHole_Pad, kbd:1pin_conn, F.Cu at (32.3, 47.4)
- added BatGND4: MountingHole_Pad, kbd:1pin_conn, F.Cu at (276.1, 47.6)
- added D0: D, kbd:D3_SMD_v2, B.Cu at (154.6, 45.2)
- added D1: D, kbd:D3_SMD_v2, B.Cu at (173.1, 48.7)
- added D10: D, kbd:D3_SMD_v2, B.Cu at (230.4, 52.4)
- added D11: D, kbd:D3_SMD_v2, B.Cu at (248.9, 54.9)
- added D12: D, kbd:D3_SMD_v2, B.Cu at (154.7, 79.3)
- added D13: D, kbd:D3_SMD_v2, B.Cu at (176.6, 87.1)
- added D14: D, kbd:D3_SMD_v2, B.Cu at (194.6, 71.7)
- added D15: D, kbd:D3_SMD_v2, B.Cu at (211.7, 64.3)
- added D16: D, kbd:D3_SMD_v2, B.Cu at (229.4, 69.8)
- added D17: D, kbd:D3_SMD_v2, B.Cu at (247.3, 71.9)
- added D18: D, kbd:D3_SMD_v2, B.Cu at (227.0, 83.8)
- added D19: D, kbd:D3_SMD_v2, B.Cu at (248.6, 86.5)
- added D2: D, kbd:D3_SMD_v2, B.Cu at (194.2, 37.0)
- added D20: D, kbd:D3_SMD_v2, B.Cu at (267.5, 93.4)
- added D3: D, kbd:D3_SMD_v2, B.Cu at (210.9, 30.8)
- added D4: D, kbd:D3_SMD_v2, B.Cu at (230.0, 34.9)
- added D5: D, kbd:D3_SMD_v2, B.Cu at (246.8, 37.4)
- added D6: D, kbd:D3_SMD_v2, B.Cu at (154.6, 62.2)
- added D7: D, kbd:D3_SMD_v2, B.Cu at (171.4, 65.7)
- added D8: D, kbd:D3_SMD_v2, B.Cu at (194.6, 54.2)
- added D9: D, kbd:D3_SMD_v2, B.Cu at (211.1, 47.2)
- added Dr0: D, kbd:D3_SMD_v2, B.Cu at (137.7, 49.3)
- added Dr1: D, kbd:D3_SMD_v2, B.Cu at (120.0, 48.1)
- added Dr10: D, kbd:D3_SMD_v2, B.Cu at (66.2, 52.3)
- added Dr11: D, kbd:D3_SMD_v2, B.Cu at (47.4, 54.6)
- added Dr12: D, kbd:D3_SMD_v2, B.Cu at (137.3, 82.5)
- added Dr13: D, kbd:D3_SMD_v2, B.Cu at (121.1, 81.4)
- added Dr14: D, kbd:D3_SMD_v2, B.Cu at (103.3, 71.0)
- added Dr15: D, kbd:D3_SMD_v2, B.Cu at (84.7, 64.1)
- added Dr16: D, kbd:D3_SMD_v2, B.Cu at (66.5, 70.3)
- added Dr17: D, kbd:D3_SMD_v2, B.Cu at (49.4, 71.2)
- added Dr18: D, kbd:D3_SMD_v2, B.Cu at (66.9, 84.1)
- added Dr19: D, kbd:D3_SMD_v2, B.Cu at (46.9, 86.3)
- added Dr2: D, kbd:D3_SMD_v2, B.Cu at (102.4, 36.6)
- added Dr20: D, kbd:D3_SMD_v2, B.Cu at (28.7, 94.7)
- added Dr3: D, kbd:D3_SMD_v2, B.Cu at (86.0, 30.4)
- added Dr4: D, kbd:D3_SMD_v2, B.Cu at (65.6, 35.9)
- added Dr5: D, kbd:D3_SMD_v2, B.Cu at (47.4, 37.9)
- added Dr6: D, kbd:D3_SMD_v2, B.Cu at (138.2, 65.9)
- added Dr7: D, kbd:D3_SMD_v2, B.Cu at (120.2, 67.0)
- added Dr8: D, kbd:D3_SMD_v2, B.Cu at (102.9, 54.4)
- added Dr9: D, kbd:D3_SMD_v2, B.Cu at (83.8, 46.8)
- added SW10_r1: SW_Push, aym1607:choc-v1-with-millmax, F.Cu at (102.4, 51.0)
- added SW13: SW_Push, aym1607:choc-v1-with-millmax, F.Cu at (247.8, 52.0)
- added SW14_r1: SW_Push, aym1607:choc-v1-with-millmax, F.Cu at (138.4, 80.0)
- added SW19: SW_Push, aym1607:choc-v1-with-millmax, F.Cu at (247.8, 69.2)
- added SW19_r1: SW_Push, aym1607:choc-v1-with-millmax, F.Cu at (48.3, 69.0)
- added SW22: SW_Push, aym1607:choc-v1-with-millmax, F.Cu at (267.8, 98.0)
- added SW22_r1: SW_Push, aym1607:choc-v1-with-millmax, F.Cu at (28.6, 97.9)
- added SW7: SW_Push, aym1607:choc-v1-with-millmax, F.Cu at (247.8, 34.9)
- added SW_POWER1: SW_SPDT, Button_Switch_SMD:SW_SPDT_PCM12, B.Cu at (26.5, 48.5)
- added SW_POWERR1: SW_SPDT, Button_Switch_SMD:SW_SPDT_PCM12, B.Cu at (270.0, 48.6)
- RSW1, RSW2: footprint kbd:SW_SPST_B3U-1000P -> kbd:ResetSW
- SW10, SW11, SW11_r1, SW12, SW12_r1, SW13_r1, SW14, SW15, SW15_r1, SW16, SW16_r1, SW17, SW17_r1, SW18, SW18_r1, SW2, SW20, SW20_r1, SW21, SW21_r1, SW2_r1, SW3, SW3_r1, SW4, SW4_r1, SW5, SW5_r1, SW6, SW6_r1, SW7_r1, SW8, SW8_r1, SW9, SW9_r1: footprint * duckyb-collection:choc-v1-with-millmax -> aym1607:choc-v1-with-millmax
- U1, U2: footprint kbd:ProMicro_v3_min -> kbd:ProMicro_v3
- moved SW13_r1 78.9 mm to (48.3, 51.9)
- moved SW7_r1 78.9 mm to (48.3, 35.0)
- moved RSW1 56.7 mm to (275.0, 85.8), turned to -90 degrees
- moved SW21 44.8 mm to (248.7, 89.4)
- moved U1 40.0 mm to (270.0, 64.3)
- moved SW9_r1 38.9 mm to (120.4, 63.0)
- moved SW15_r1 38.9 mm to (120.4, 80.0)
- moved SW17_r1 37.4 mm to (84.4, 61.1)
- moved SW18_r1 36.7 mm to (66.3, 66.4)
- moved SW8_r1 36.7 mm to (138.4, 63.0)
- moved REF** 36.1 mm to (221.3, 42.9)
- moved SW16_r1 35.8 mm to (102.4, 68.0)
- moved SW20_r1 32.1 mm to (68.1, 86.4), turned to 180 degrees
- moved RSW2 21.0 mm to (21.3, 85.5), turned to 90 degrees
- moved SW5 20.0 mm to (211.8, 27.0)
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Connections:
- RSW2 pad 1: gnd -> gnd_r
- SW10 pad 1: Switch8 -> col2
- SW10 pad 2: gnd -> Net-(D8-Pad2)
- SW11 pad 1: Switch9 -> col3
- SW11 pad 2: gnd -> Net-(D9-Pad2)
- SW11_r1 pad 1: Switch9_r -> col3r
- SW11_r1 pad 2: gnd -> Net-(SW11_r1-Pad2)
- SW12 pad 1: Switch10 -> col4
- SW12 pad 2: gnd -> Net-(D10-Pad2)
- SW12_r1 pad 1: Switch10_r -> col4r
- SW12_r1 pad 2: gnd -> Net-(Dr10-Pad2)
- SW13_r1 pad 1: Switch11_r -> col5r
- SW13_r1 pad 2: gnd -> Net-(Dr11-Pad2)
- SW14 pad 1: Switch11 -> col0
- SW14 pad 2: gnd -> Net-(D12-Pad2)
- SW15 pad 1: Switch12 -> col1
- SW15 pad 2: gnd -> Net-(D13-Pad2)
- SW15_r1 pad 1: Switch13_r -> col1r
- SW15_r1 pad 2: gnd -> Net-(Dr13-Pad2)
- SW16 pad 1: Switch13 -> col2
- SW16 pad 2: gnd -> Net-(D14-Pad2)
- SW16_r1 pad 1: Switch14_r -> col2r
- SW16_r1 pad 2: gnd -> Net-(SW16_r1-Pad2)
- SW17 pad 1: Switch14 -> col3
- SW17 pad 2: gnd -> Net-(D15-Pad2)
- SW17_r1 pad 1: Switch15_r -> col3r
- SW17_r1 pad 2: gnd -> Net-(SW17_r1-Pad2)
- SW18 pad 1: Switch15 -> col4
- SW18 pad 2: gnd -> Net-(D16-Pad2)
- SW18_r1 pad 1: Switch12_r -> col4r
- SW18_r1 pad 2: gnd -> Net-(SW18_r1-Pad2)
- SW2 pad 1: Switch1 -> col0
- SW2 pad 2: gnd -> Net-(D0-Pad2)
- SW20 pad 1: Switch17 -> col3
- SW20 pad 2: gnd -> Net-(D18-Pad2)
- SW20_r1 pad 1: Switch17_r -> col3r
- SW20_r1 pad 2: gnd -> Net-(Dr18-Pad2)
- SW21 pad 1: Switch16 -> col4
- SW21 pad 2: gnd -> Net-(D19-Pad2)
- SW21_r1 pad 1: Switch16_r -> col4r
- SW21_r1 pad 2: gnd -> Net-(SW21_r1-Pad2)
- SW2_r1 pad 1: Switch1_r -> col0r
- SW2_r1 pad 2: gnd -> Net-(Dr0-Pad2)
- SW3 pad 1: Switch2 -> col1
- SW3 pad 2: gnd -> Net-(D1-Pad2)
- SW3_r1 pad 1: Switch2_r -> col1r
- SW3_r1 pad 2: gnd -> Net-(SW3_r1-Pad2)
- SW4 pad 1: Switch3 -> col2
- SW4 pad 2: gnd -> Net-(D2-Pad2)
- SW4_r1 pad 1: Switch3_r -> col2r
- SW4_r1 pad 2: gnd -> Net-(Dr2-Pad2)
- SW5 pad 1: Switch4 -> col3
- SW5 pad 2: gnd -> Net-(D3-Pad2)
- SW5_r1 pad 1: Switch4_r -> col3r
- SW5_r1 pad 2: gnd -> Net-(SW5_r1-Pad2)
- SW6 pad 1: Switch5 -> col4
- SW6 pad 2: gnd -> Net-(D4-Pad2)
- SW6_r1 pad 1: Switch5_r -> col4r
- SW6_r1 pad 2: gnd -> Net-(Dr4-Pad2)
- SW7_r1 pad 1: Switch6_r -> col5r
- SW7_r1 pad 2: gnd -> Net-(Dr5-Pad2)
- SW8 pad 1: Switch6 -> col0
- SW8 pad 2: gnd -> Net-(D6-Pad2)
- SW8_r1 pad 1: Switch7_r -> col0r
- SW8_r1 pad 2: gnd -> Net-(SW8_r1-Pad2)
- SW9 pad 1: Switch7 -> col1
- SW9 pad 2: gnd -> Net-(D7-Pad2)
- SW9_r1 pad 1: Switch8_r -> col1r
- SW9_r1 pad 2: gnd -> Net-(SW9_r1-Pad2)
- U1 pad 1: Switch10 -> unconnected-(U1-Pad1)
- U1 pad 10: Switch1 -> row_3
- U1 pad 11: Switch16 -> unconnected-(U1-Pad11)
- U1 pad 12: Switch17 -> unconnected-(U1-Pad12)
- U1 pad 13: Switch9 -> unconnected-(U1-Pad13)
- U1 pad 14: Switch8 -> unconnected-(U1-Pad14)
- U1 pad 15: Switch7 -> col5
- U1 pad 16: Switch6 -> col4
- U1 pad 17: Switch2 -> col3
- U1 pad 18: Switch3 -> col2
- U1 pad 19: Switch4 -> col1
- U1 pad 2: Switch18 -> unconnected-(U1-Pad2)
- U1 pad 20: Switch5 -> col0
- U1 pad 5: Switch11 -> unconnected-(U1-Pad5)
- U1 pad 6: Switch12 -> unconnected-(U1-Pad6)
- U1 pad 7: Switch13 -> row_0
- U1 pad 8: Switch14 -> row_1
- U1 pad 9: Switch15 -> row_2
- U2 pad 1: Switch10_r -> unconnected-(U2-Pad1)
- U2 pad 10: Switch1_r -> row_3r
- U2 pad 11: Switch16_r -> unconnected-(U2-Pad11)
- U2 pad 12: Switch17_r -> unconnected-(U2-Pad12)
- U2 pad 13: Switch9_r -> unconnected-(U2-Pad13)
- U2 pad 14: Switch8_r -> unconnected-(U2-Pad14)
- U2 pad 15: Switch7_r -> col5r
- U2 pad 16: Switch6_r -> col4r
- U2 pad 17: Switch2_r -> col3r
- U2 pad 18: Switch3_r -> col2r
- U2 pad 19: Switch4_r -> col1r
- U2 pad 2: Switch18_r -> unconnected-(U2-Pad2)
- U2 pad 20: Switch5_r -> col0r
- U2 pad 21: vcc -> vcc_r
- U2 pad 23: gnd -> gnd_r
- U2 pad 24: raw -> raw_r
- U2 pad 3: gnd -> gnd_r
- U2 pad 4: gnd -> gnd_r
- U2 pad 5: Switch11_r -> unconnected-(U2-Pad5)
- U2 pad 6: Switch12_r -> unconnected-(U2-Pad6)
- U2 pad 7: Switch13_r -> row_0r
- U2 pad 8: Switch14_r -> row_1r
- U2 pad 9: Switch15_r -> row_2r
Routing:
- net Switch6_r: track 135.8 -> 0.00 mm
- net Switch11: track 131.7 -> 0.00 mm
- net Switch1: track 130.7 -> 0.00 mm, vias 1 -> 0
- net Switch1_r: track 119.7 -> 0.00 mm, vias 1 -> 0
- net Switch7_r: track 111.0 -> 0.00 mm
- net Switch2_r: track 110.1 -> 0.00 mm
- net Switch12: track 108.7 -> 0.00 mm
- net Switch6: track 107.4 -> 0.00 mm
- net Switch11_r: track 100.0 -> 0.00 mm
- net Switch3_r: track 91.8 -> 0.00 mm
- net Switch13: track 90.4 -> 0.00 mm
- net Switch8_r: track 89.9 -> 0.00 mm
- net Switch2: track 89.9 -> 0.00 mm
- net Switch7: track 84.6 -> 0.00 mm
- net Switch4_r: track 72.6 -> 0.00 mm
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- removed copper zone on B.Cu, net gnd
- removed copper zone on F.Cu, net gnd
Other:
- board size 216.9 x 86.9 mm -> 261.1 x 90.8 mm
- board text removed: "Sweep is based on the Ferris."
- board text removed: "Sweep v 2.2"

Commit message: Done with routing.
Parts:
- moved BatGND4 243.9 mm to (32.2, 47.6)
- moved Bat+r1 243.9 mm to (20.0, 47.6)
- moved SW_POWERR1 243.8 mm to (26.2, 48.5)
- moved BatGND1 243.7 mm to (276.0, 47.4)
- moved SW_POWER1 243.4 mm to (269.9, 48.7)
- moved Bat+1 243.2 mm to (263.9, 47.4)
- moved D13 10.8 mm to (175.9, 76.3)
- moved D20 9.58 mm to (264.6, 102.6), turned to 145 degrees
- moved D18 8.61 mm to (228.5, 92.3)
- moved Dr19 8.61 mm to (49.3, 94.6), turned to -165 degrees
- moved Dr20 8.32 mm to (31.9, 102.4), turned to -145 degrees
- moved D19 8.31 mm to (247.3, 94.7), turned to 165 degrees
- moved Dr16 7.95 mm to (66.3, 62.4), turned to 0 degrees
- moved Dr18 7.95 mm to (68.2, 91.9)
- moved D7 7.86 mm to (175.7, 59.1)
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Routing:
- net row_0: track 0.00 -> 213.1 mm
- net row_1: track 0.00 -> 188.3 mm
- net col0r: track 0.00 -> 186.0 mm, vias 0 -> 3
- net row_0r: track 0.00 -> 174.3 mm, vias 0 -> 4
- net row_2: track 0.00 -> 171.9 mm
- net col0: track 0.00 -> 162.3 mm, vias 0 -> 3
- net col1r: track 0.00 -> 158.9 mm, vias 0 -> 2
- net row_1r: track 0.00 -> 148.3 mm
- net col1: track 0.00 -> 141.6 mm, vias 0 -> 2
- net col2r: track 1.18 -> 137.4 mm, vias 0 -> 1
- net row_2r: track 0.00 -> 135.4 mm
- net col2: track 0.49 -> 124.6 mm, vias 0 -> 1
- net col3r: track 0.70 -> 121.2 mm, vias 0 -> 1
- net col3: track 0.00 -> 110.0 mm, vias 0 -> 1
- net col4r: track 0.00 -> 99.5 mm, vias 0 -> 1
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Other:
- board size 261.1 x 90.8 mm -> 261.1 x 90.7 mm
