File: Swept/sweepv2.kicad_pcb (KiCad board)
At the start: 2 copper layers, 261.1 x 90.7 mm, 98 parts, among them SW10 SW_Push, SW10_r1 SW_Push, SW11 SW_Push, SW11_r1 SW_Push, SW12 SW_Push, SW12_r1 SW_Push, SW13 SW_Push, SW13_r1 SW_Push, SW14 SW_Push, SW14_r1 SW_Push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

Commit message: Create version 0.1.2
Parts:
- renumbered Bat+1 to +, Bat+r1 to +, BatGND1 to -, BatGND4 to -
