File: Swept/sweepv2.kicad_sch (KiCad schematic)
At the start: 94 parts, among them SW10 SW_Push, SW10_r1 SW_Push, SW11 SW_Push, SW11_r1 SW_Push, SW12 SW_Push, SW12_r1 SW_Push, SW13 SW_Push, SW13_r1 SW_Push, SW14 SW_Push, SW14_r1 SW_Push, SW15 SW_Push, SW15_r1 SW_Push, SW16 SW_Push, SW16_r1 SW_Push, SW17 SW_Push, SW17_r1 SW_Push, SW18 SW_Push, SW18_r1 SW_Push, SW19 SW_Push, SW19_r1 SW_Push, SW2 SW_Push, SW20 SW_Push, SW20_r1 SW_Push, SW21 SW_Push, SW21_r1 SW_Push, SW22 SW_Push, SW22_r1 SW_Push, SW2_r1 SW_Push, SW3 SW_Push, SW3_r1 SW_Push, SW4 SW_Push, SW4_r1 SW_Push, SW5 SW_Push, SW5_r1 SW_Push, SW6 SW_Push, SW6_r1 SW_Push, SW7 SW_Push, SW7_r1 SW_Push, SW8 SW_Push, SW8_r1 SW_Push, SW9 SW_Push, SW9_r1 SW_Push, U1 ProMicro-kbd, U2 ProMicro-kbd

Commit message: Done with routing.
Parts:
- Dr0, Dr1, Dr10, Dr11, Dr12, Dr13, Dr14, Dr15, Dr16, Dr17, Dr18, Dr19, Dr2, Dr20, Dr3, Dr4, Dr5, Dr6, Dr7, Dr8, Dr9: value 1N4448W -> D
Connections:
- net col5: now also SW22.1
- net col0r: now reaches SW2_r1.1
- net col0r: now also SW14_r1.1, SW8_r1.1, U2.20 (F4)
- net at SW2_r1.2: now also Dr0.2 (A)
- net col1r: now reaches SW3_r1.1
- net col1r: now also SW15_r1.1, SW9_r1.1, U2.19 (F5)
- net at SW3_r1.2: now also Dr1.2 (A)
- net col2r: now reaches SW4_r1.1
- net col2r: now also SW10_r1.1, SW16_r1.1, U2.18 (F6)
- net at SW4_r1.2: now also Dr2.2 (A)
- net col3r: now reaches SW5_r1.1
- net col3r: now also SW11_r1.1, SW17_r1.1, SW20_r1.1, U2.17 (F7)
- net at SW5_r1.2: now also Dr3.2 (A)
- net col4r: now reaches SW6_r1.1
- net col4r: now also SW12_r1.1, SW18_r1.1, SW21_r1.1, U2.16 (B1)
- net at SW6_r1.2: now also Dr4.2 (A)
- net at SW17_r1.2: now also Dr15.2 (A)
- net at SW18_r1.2: now also Dr16.2 (A)
- net col5r: now reaches SW7_r1.1
- net col5r: now also SW13_r1.1, SW19_r1.1, SW22_r1.1, U2.15 (B3)
- net at SW7_r1.2: now also Dr5.2 (A)
- net at SW8_r1.2: now also Dr6.2 (A)
- net at SW9_r1.2: now also Dr7.2 (A)
- net at SW10_r1.2: now also Dr8.2 (A)
- net at SW11_r1.2: now also Dr9.2 (A)
- net at SW12_r1.2: now also Dr10.2 (A)
- net at SW13_r1.2: now also Dr11.2 (A)
- net at SW14_r1.2: now also Dr12.2 (A)
- net at SW15_r1.2: now also Dr13.2 (A)
- net at SW16_r1.2: now also Dr14.2 (A)
- net row_3r: now reaches U2.10 (E6)
- net row_3r: now also Dr18.1 (K), Dr19.1 (K), Dr20.1 (K)
- net row_0r: now reaches U2.7 (D4)
- net row_0r: now also Dr0.1 (K), Dr1.1 (K), Dr2.1 (K), Dr3.1 (K), Dr4.1 (K), Dr5.1 (K)
- net row_1r: now reaches U2.8 (C6)
- net row_1r: now also Dr10.1 (K), Dr11.1 (K), Dr6.1 (K), Dr7.1 (K), Dr8.1 (K), Dr9.1 (K)
- net row_2r: now reaches U2.9 (D7)
- net row_2r: now also Dr12.1 (K), Dr13.1 (K), Dr14.1 (K), Dr15.1 (K), Dr16.1 (K), Dr17.1 (K)
- net at Dr20.2 (A): now also SW22_r1.2
- net at Dr18.2 (A): now also SW20_r1.2
- net at Dr19.2 (A): now also SW21_r1.2
- net at SW19_r1.2: now also Dr17.2 (A)
- no-connect marks 8 -> 16
Other:
- moved on the sheet: Dr8
