File: Swept_3x6/Swept_3x6.kicad_pcb (KiCad board)
At the start: 2 copper layers, 261.1 x 90.7 mm, 98 parts, among them SW10 SW_Push, SW10_r1 SW_Push, SW11 SW_Push, SW11_r1 SW_Push, SW12 SW_Push, SW12_r1 SW_Push, SW13 SW_Push, SW13_r1 SW_Push, SW14 SW_Push, SW14_r1 SW_Push, SW15 SW_Push, SW15_r1 SW_Push, SW16 SW_Push, SW16_r1 SW_Push, SW17 SW_Push, SW17_r1 SW_Push, SW18 SW_Push, SW18_r1 SW_Push, SW19 SW_Push, SW19_r1 SW_Push, SW2 SW_Push, SW20 SW_Push, SW20_r1 SW_Push, SW21 SW_Push, SW21_r1 SW_Push, SW22 SW_Push, SW22_r1 SW_Push, SW2_r1 SW_Push, SW3 SW_Push, SW3_r1 SW_Push, SW4 SW_Push, SW4_r1 SW_Push, SW5 SW_Push, SW5_r1 SW_Push, SW6 SW_Push, SW6_r1 SW_Push, SW7 SW_Push, SW7_r1 SW_Push, SW8 SW_Push, SW8_r1 SW_Push, SW9 SW_Push, SW9_r1 SW_Push, U1 ProMicro-kbd, U2 ProMicro-kbd

Commit message: Added support for Kailh hot-swap sockets.
Parts:
- SW10, SW10_r1, SW11, SW11_r1, SW12, SW12_r1, SW13, SW13_r1, SW14, SW14_r1, SW15, SW15_r1, SW16, SW16_r1, SW17, SW17_r1, SW18, SW18_r1, SW19, SW19_r1, SW2, SW20, SW20_r1, SW21, SW21_r1, SW22, SW22_r1, SW2_r1, SW3, SW3_r1, SW4, SW4_r1, SW5, SW5_r1, SW6, SW6_r1, SW7, SW7_r1, SW8, SW8_r1, SW9, SW9_r1: footprint aym1607:choc-v1-with-millmax -> keyswitches:Kailh_socket_PG1350_optional
- moved Dr20 16.6 mm to (29.4, 86.1)
- moved D18 11.0 mm to (223.2, 82.7)
- moved D8 10.4 mm to (198.9, 56.3)
- moved D17 10.3 mm to (253.0, 74.2)
- moved D16 10.3 mm to (234.5, 71.9)
- moved D15 10.2 mm to (216.5, 66.4)
- moved D11 10.0 mm to (252.3, 57.1)
- moved D5 10.0 mm to (252.5, 39.9)
- moved D19 9.99 mm to (245.1, 84.9)
- moved D13 9.95 mm to (181.0, 84.9)
- moved D6 9.87 mm to (162.4, 67.9)
- moved Dr19 9.85 mm to (43.5, 86.6)
- moved D1 9.82 mm to (181.3, 50.1)
- moved D4 9.81 mm to (234.5, 37.2)
- moved D20 9.80 mm to (265.3, 92.8)
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- renumbered + to Bat+1, + to Bat+r1, - to BatGND1, - to BatGND4
Routing:
- net col3: track 110.0 -> 161.3 mm, vias 1 -> 5
- net col3r: track 121.2 -> 172.3 mm, vias 1 -> 5
- net col4r: track 99.5 -> 149.1 mm, vias 1 -> 4
- net col5r: track 94.0 -> 143.4 mm, vias 0 -> 7
- net col1: track 141.6 -> 183.6 mm, vias 2 -> 4
- net col4: track 86.1 -> 127.7 mm, vias 1 -> 5
- net col1r: track 158.9 -> 198.7 mm, vias 2 -> 4
- net col0: track 162.3 -> 201.8 mm, vias 3 -> 5
- net col2r: track 137.4 -> 175.6 mm, vias 1 -> 5
- net col2: track 124.6 -> 160.5 mm, vias 1 -> 4
- net col5: track 98.6 -> 131.6 mm, vias 0 -> 4
- net col0r: track 186.0 -> 215.4 mm, vias 3 -> 5
- net row_0r: track 174.3 -> 145.9 mm, vias 4 -> 0
- net row_2: track 171.9 -> 147.7 mm
- net row_1r: track 148.3 -> 168.5 mm
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Other:
- outline, holes or cut-outs redrawn

Commit message: Added nice!view suppor for 3x6
Parts:
- added J1: ScreenL, Connector_PinHeader_2.54mm:PinHeader_1x05_P2.54mm_Vertical, F.Cu at (265.0, 82.2)
- added J2: ScreenR, Connector_PinHeader_2.54mm:PinHeader_1x05_P2.54mm_Vertical, F.Cu at (21.2, 82.1)
- moved Dr20 9.08 mm to (37.3, 90.5), turned to -55 degrees
- moved RSW1 4.46 mm to (274.2, 90.1), turned to -35 degrees
- moved RSW2 4.29 mm to (23.8, 89.0), turned to 35 degrees
Connections:
- U1 pad 1: unconnected-(U1-Pad1) -> CS
- U1 pad 5: unconnected-(U1-Pad5) -> MOSI
- U1 pad 6: unconnected-(U1-Pad6) -> SCK
- U2 pad 1: unconnected-(U2-Pad1) -> CSr
- U2 pad 5: unconnected-(U2-Pad5) -> MOSIr
- U2 pad 6: unconnected-(U2-Pad6) -> SCKr
Routing:
- net vcc_r: track 0.00 -> 52.2 mm
- net CSr: track 0.00 -> 37.3 mm, vias 0 -> 1
- net CS: track 0.00 -> 35.4 mm, vias 0 -> 1
- net MOSIr: track 0.00 -> 31.5 mm
- net MOSI: track 0.00 -> 31.2 mm
- net vcc: track 0.00 -> 27.9 mm, vias 0 -> 1
- net SCKr: track 0.00 -> 27.7 mm
- net SCK: track 0.00 -> 27.6 mm
- net gnd: track 53.5 -> 73.2 mm, vias 0 -> 1
- net gnd_r: track 68.0 -> 86.2 mm
- net row_3r: track 63.6 -> 51.0 mm
- net reset_r: track 28.5 -> 39.0 mm
- net col3r: track 172.3 -> 182.5 mm
- net col4r: track 149.1 -> 158.3 mm
- net reset: track 41.8 -> 37.1 mm, vias 0 -> 1
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
Commit message: Version 1.1.1 of the 3x6 swept.
Parts:
- added ?: , , F.Cu at (166.8, 54.6)
- added ?: , , F.Cu at (84.1, 79.5)
- added ?: , , F.Cu at (166.8, 71.6)
- added ?: , , F.Cu at (212.4, 79.2)
- added ?: , , F.Cu at (129.3, 54.6)
- added ?: , , F.Cu at (257.8, 60.6)
- added ?: , , F.Cu at (37.5, 91.6)
- added ?: , , F.Cu at (129.3, 71.5)
- added ?: , , F.Cu at (258.6, 92.0)
- added ?: , , F.Cu at (38.5, 60.3)
- moved Dr20 6.60 mm to (32.2, 86.3), turned to 0 degrees
Routing:
- net row_3r: track 51.0 -> 58.3 mm
- net col3: track 161.3 -> 157.7 mm
- net gnd_r: track 86.2 -> 83.2 mm
- net BT+_r: track 12.9 -> 10.7 mm
- net col5r: track 143.8 -> 145.6 mm
- net Net-(Dr20-Pad2): track 21.9 -> 23.7 mm
- net raw_r: track 15.2 -> 14.0 mm
- net raw: track 14.2 -> 15.1 mm
- net row_1r: track 168.5 -> 167.6 mm
- net gnd: track 73.2 -> 73.8 mm
- net row_2: track 148.1 -> 147.5 mm
